File: lopafi/lopafi1.sch (KiCad schematic (older format))
At the start: 37 parts

Commit message: first schematic
Parts:
- added C12: 100n, symbol C_Small
- added J1, J2: Conn_01x01, symbol Conn_01x01
- added J3: Conn_02x03_Odd_Even, symbol Conn_02x03_Odd_Even
- added J4: Conn_02x20_Odd_Even, symbol Conn_02x20_Odd_Even
- added J5, J6: Conn_Coaxial, symbol Conn_Coaxial
- added R1, R2, R3, R4, R5, R6: 4k7, symbol R_Small
- added U1: TCA9534, symbol TCA9534
- gave numbers to parts that had none: 37
Connections:
- net +5V: now also C12.2, J3.1 (Pin_1), J3.3 (Pin_3), J3.5 (Pin_5), J4.2 (Pin_2), J4.4 (Pin_4), R1.1, R2.1, R3.1, U1.16 (VDD)
- net 12MHz: now also U1.6 (P2)
- net 2.5MHz: now also U1.4 (P0)
- net 6MHz: now also U1.5 (P1)
- net GND: now also C12.1, J1.1 (Pin_1), J2.1 (Pin_1), J4.14 (Pin_14), J4.20 (Pin_20), J4.25 (Pin_25), J4.30 (Pin_30), J4.34 (Pin_34), J4.39 (Pin_39), J4.6 (Pin_6), J4.9 (Pin_9), R4.2, R5.2, R6.2, U1.8 (GND)
- new net: J4.32 (Pin_32), J5.1 (In), J6.1 (In)
- new net: R3.2, U1.13 (~INT~)
- new net: J3.2 (Pin_2), R4.1, U1.1 (A0)
- new net: J3.4 (Pin_4), R5.1, U1.2 (A1)
- new net: J3.6 (Pin_6), R6.1, U1.3 (A2)
- new net: J5.2 (Ext), J6.2 (Ext)
- new net SCL: J4.5 (Pin_5), R1.2, U1.14 (SCL)
- new net SDA: J4.3 (Pin_3), R2.2, U1.15 (SDA)
- no-connect marks 0 -> 32
Other:
- note added: "(envisager de coller une liaison coax entre gpio et connecteur situé du coté opposé de la carte)"
- note added: "2.6 mm fixing holes"
- note added: "RF OUT\n"
- moved on the sheet: C1, C10, C11, C13, C14, C15, C16, C17, C18, C19, C2, C20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
